File: kicadFiles/doddle60.kicad_pcb (KiCad board)
At the start: 2 copper layers, 283 x 94.2 mm, 198 parts, among them J1 TYPE-C-31-M12_13, J2 Conn_01x14, J3 Conn_ARM_JTAG_SWD_10, SW1 ESC, SW10 9, SW11 0, SW12 -_, SW13 +=, SW14 2U BKSP, SW15 TAB_150, SW16 Q, SW17 W, SW18 E, SW19 R, SW2 1, SW20 T, SW21 Y, SW22 U, SW23 I, SW24 O, SW25 P, SW26 [{, SW27 ]}, SW28 1U_RBKSP, SW29 CAPS_175, SW3 2, SW30 A, SW31 S, SW32 D, SW33 F, SW34 G, SW35 H, SW36 J, SW37 K, SW38 L, SW39 :;, SW4 3, SW40 @', SW41 ~~#, SW42 LSHIFT_125, SW43 |\, SW44 Z, SW45 X, SW46 C, SW47 V, SW48 B, SW49 N, SW5 4, SW50 M, SW51 <,, SW52 >., SW53 ?/, SW54 LCTRL_150, SW55 LGUI_100, SW56 LALT_150, SW57 SPACE_700, SW58 RALT_150, SW59 RGUI_100, SW6 5, SW60 RCTRL_150, SW61 LCTRL_125, SW62 LGUI_125, SW63 STEPPED_CAPS_125, SW64 1U LBKSP, SW65 ISO_Enter, SW66 LALT_125, SW67 SPACE_625, SW68 RALT_125, SW69 RGUI_125, SW7 6, SW70 FN_125, SW71 RCTRL_125, SW72 RSHIFT_275, SW73 LSHIFT_225, SW74 RSHIFT_175, SW75 FN_100, SW8 7, SW9 8, U1 STM32F072-LQFP48, U2 USBLC6-2SC6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

Commit message: PCB1
Parts:
- removed the SW62 at (320.0, 167.6)
- added D64: 1N4148, acheron_Components:D_SOD-123, F.Cu at (288.8, 163.4)
- added D66: 1N4148, acheron_Components:D_SOD-123, F.Cu at (203.4, 161.7)
- added D67: 1N4148, acheron_Components:D_SOD-123, F.Cu at (184.4, 161.4)
- added D68: 1N4148, acheron_Components:D_SOD-123, F.Cu at (93.4, 104.8)
- added SW66: SPACE_275, acheron_MX_SolderMask:MX275R, F.Cu at (258.1, 167.5)
- added SW76: 150U_BKSLH, acheron_MX_SolderMask:MX150, F.Cu at (84.2, 110.4)
- added SW77: ANSI_Enter, acheron_MX_SolderMask:MX225R, F.Cu at (112.9, 129.4)
- added SW78: BKSLSH_1U, acheron_MX_SolderMask:MX100, F.Cu at (112.8, 148.5)
- added SW79: RSHIFT_1.75, acheron_MX_SolderMask:MX175, F.Cu at (86.6, 148.5)
- added SW80: HENKAN_125, acheron_MX_SolderMask:MX125, F.Cu at (172.4, 167.6)
- added SW81: MUHENKAN_125, acheron_MX_SolderMask:MX125, F.Cu at (272.4, 167.6)
- added SW82: RALT_125, acheron_MX_SolderMask:MX125, F.Cu at (148.6, 167.6)
- added SW83: RALT_125, acheron_MX_SolderMask:MX125, F.Cu at (124.8, 167.6)
- added SW84: RGUI_100, acheron_MX_SolderMask:MX100, F.Cu at (103.4, 167.6)
- added SW85: RCTRL_125, acheron_MX_SolderMask:MX125, F.Cu at (81.9, 167.6)
- added SW86: KANA_100, acheron_MX_SolderMask:MX100, F.Cu at (174.8, 167.5)
- added SW89: HENKAN_125, acheron_MX_SolderMask:MX125, F.Cu at (196.2, 167.5)
- SW54: value LCTRL_150 -> LCTRL_125; footprint acheron_MX_SolderMask:MX150 -> acheron_MX_SolderMask:MX125
- SW55: value LGUI_100 -> LGUI_125; footprint acheron_MX_SolderMask:MX100 -> acheron_MX_SolderMask:MX125
- SW56: value LALT_150 -> LALT_125; footprint acheron_MX_SolderMask:MX150 -> acheron_MX_SolderMask:MX125
- SW57: value SPACE_700 -> SPACE_275; footprint acheron_MX_SolderMask:MX700R -> acheron_MX_SolderMask:MX275R
- SW58: value RALT_150 -> RALT_125; footprint acheron_MX_SolderMask:MX150 -> acheron_MX_SolderMask:MX125
- SW59: value RGUI_100 -> RGUI_125; footprint acheron_MX_SolderMask:MX100 -> acheron_MX_SolderMask:MX125
- SW60: value RCTRL_150 -> RCTRL_125; footprint acheron_MX_SolderMask:MX150 -> acheron_MX_SolderMask:MX125
- SW61: value LCTRL_125 -> LGUI_100; footprint acheron_MX_SolderMask:MX125 -> acheron_MX_SolderMask:MX100
- SW67: value SPACE_625 -> MUHENKAN_100; footprint acheron_MX_SolderMask:MX625R -> acheron_MX_SolderMask:MX100
- SW69: value RGUI_125 -> SPACE_125
- SW70: value FN_125 -> SPACE_450; footprint acheron_MX_SolderMask:MX125 -> acheron_MX_SolderMask:MX100
- SW71: value RCTRL_125 -> SPACE_225; footprint acheron_MX_SolderMask:MX125 -> acheron_MX_SolderMask:MX225R
- SW72: footprint acheron_MX_SolderMask:MX275 -> acheron_MX_SolderMask:MX275R
- SW73: footprint acheron_MX_SolderMask:MX225 -> acheron_MX_SolderMask:MX225R
- moved G2 206.1 mm to (386.9, 221.1)
- moved G1 157.8 mm to (391.4, 237.4)
- moved G4 157.7 mm to (378.8, 259.9)
- moved G5 157.7 mm to (378.8, 259.9)
- moved SW70 121.5 mm to (227.2, 167.6)
- moved SW71 104.8 mm to (186.6, 167.6)
- moved SW69 90.5 mm to (220.0, 167.6)
- moved SW67 54.9 mm to (279.6, 167.6)
- moved D57 49.0 mm to (252.3, 160.9)
- moved SW57 21.5 mm to (234.3, 167.6)
- moved SW54 19.0 mm to (322.4, 167.6)
- moved SW56 7.24 mm to (301.0, 167.7)
- moved J3 3.28 mm to (310.5, 167.6)
- moved SW55 2.46 mm to (320.1, 167.6)
- moved SW60 2.38 mm to (81.9, 167.6)
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- renumbered SW66 to SW62
Connections:
- SW54 pad 1: Col1 -> Col2
- SW54 pad 2: Net-(D54-Pad2) -> Net-(D55-Pad2)
- SW57 pad 1: Col10 -> Col7
- SW67 pad 1: Col10 -> Col4
- SW67 pad 2: Net-(D57-Pad2) -> Net-(D64-Pad2)
- SW69 pad 1: Col12 -> Net-(SW69-Pad1)
- SW69 pad 2: Net-(D58-Pad2) -> Net-(D57-Pad2)
- SW70 pad 1: Col13 -> Net-(SW69-Pad1)
- SW70 pad 2: Net-(D59-Pad2) -> Net-(D57-Pad2)
- SW71 pad 1: Col14 -> Col8
- SW71 pad 2: Net-(D60-Pad2) -> Net-(D66-Pad2)
- U1 pad 41: Extra1 -> Col15
Routing:
- net Net-(D66-Pad2): track 0.00 -> 28.1 mm
- net Net-(D57-Pad2): track 28.1 -> 0.00 mm
- net Col10: track 548.5 -> 536.8 mm
- net Net-(SW69-Pad1): track 0.00 -> 11.7 mm
- net Col3: track 215.5 -> 212.3 mm
- net Net-(D55-Pad2): track 12.4 -> 10.1 mm
- net Col2: track 138.7 -> 136.5 mm

Commit message: PCB
Parts:
- moved G3 192.4 mm to (353.6, 244.4)
Changed lines of the file:
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@@
   )
   (module acheron_Logos:acheronLong (layer F.Cu)
-    (at 209.254375 117.134125)
+    (at 353.61337 244.365265)
     (fp_text reference G3 (at 0 0) (layer F.SilkS) hide
       (effects (font (size 1.524 1.524) (thickness 0.3)))

Commit message: cache
Parts:
- removed SW66: SPACE_275, acheron_MX_SolderMask:MX275R
- removed SW69: SPACE_125, acheron_MX_SolderMask:MX125
- removed SW71: SPACE_225, acheron_MX_SolderMask:MX225R
- removed SW85: RCTRL_125, acheron_MX_SolderMask:MX125
- SW70: footprint acheron_MX_SolderMask:MX100 -> acheron_MX_SolderMask:MX450R
- SW77: footprint acheron_MX_SolderMask:MX225R -> acheron_MX_SolderMask:MX225
- moved D56 7.36 mm to (289.2, 161.6)
- moved D67 3.72 mm to (180.7, 161.0)
- moved D64 3.02 mm to (286.3, 161.6)
- moved RRST1 2.50 mm to (257.1, 150.1)
- moved CRST2 2.33 mm to (249.2, 150.4)
- moved D62 1.62 mm to (113.6, 143.7)
- moved CRST1 1.22 mm to (259.8, 151.4)
- moved QRST1 1.16 mm to (251.9, 151.4)
- turned J3 to 180 degrees
Connections:
- SW70 pad 1: Net-(SW69-Pad1) -> Col7
- SW80 pad 1: Col8 -> Col9
- SW80 pad 2: Net-(D66-Pad2) -> Net-(D67-Pad2)
- SW86 pad 1: Col9 -> Col8
- SW86 pad 2: Net-(D67-Pad2) -> Net-(D66-Pad2)
Routing:
- net Col15: track 0.00 -> 267.7 mm, vias 0 -> 3
- net Col7: track 380.7 -> 583.4 mm
- net Col8: track 391.2 -> 575.0 mm
- net Col10: track 536.8 -> 369.2 mm
- net GND: track 0.63 -> 153.1 mm, vias 2 -> 11
- net Col9: track 373.4 -> 513.1 mm
- net Col4: track 213.0 -> 311.3 mm
- net Extra1: track 38.9 -> 0.00 mm
- net Net-(D65-Pad2): track 15.0 -> 52.6 mm, vias 0 -> 1
- net Col14: track 358.6 -> 388.4 mm
- net Net-(D57-Pad2): track 0.00 -> 22.5 mm
- net Col13: track 336.1 -> 348.2 mm
- net Net-(D64-Pad2): track 0.00 -> 12.0 mm
- net Col3: track 212.3 -> 224.1 mm, vias 0 -> 1
- net Net-(SW69-Pad1): track 11.7 -> 0.00 mm
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Other:
- outline, holes or cut-outs redrawn
