File: kicadFiles/doddle60.sch (KiCad schematic (older format))
At the start: 198 parts, among them J1 TYPE-C-31-M12_13, J2 Conn_01x14, J3 Conn_ARM_JTAG_SWD_10, SW1 ESC, SW10 9, SW11 0, SW12 -_, SW13 +=, SW14 2U BKSP, SW15 TAB_150, SW16 Q, SW17 W, SW18 E, SW19 R, SW2 1, SW20 T, SW21 Y, SW22 U, SW23 I, SW24 O, SW25 P, SW26 [{, SW27 ]}, SW28 1U_RBKSP, SW29 CAPS_175, SW3 2, SW30 A, SW31 S, SW32 D, SW33 F, SW34 G, SW35 H, SW36 J, SW37 K, SW38 L, SW39 :;, SW4 3, SW40 @', SW41 ~~#, SW42 LSHIFT_125, SW43 |\\, SW44 Z, SW45 X, SW46 C, SW47 V, SW48 B, SW49 N, SW5 4, SW50 M, SW51 <,, SW52 >., SW53 ?/, SW54 LCTRL_150, SW55 LGUI_100, SW56 LALT_150, SW57 SPACE_700, SW58 RALT_150, SW59 RGUI_100, SW6 5, SW60 RCTRL_150, SW61 LCTRL_125, SW62 LGUI_125, SW63 STEPPED_CAPS_125, SW64 1U LBKSP, SW65 ISO_Enter, SW66 LALT_125, SW67 SPACE_625, SW68 RALT_125, SW69 RGUI_125, SW7 6, SW70 FN_125, SW71 RCTRL_125, SW72 RSHIFT_275, SW73 LSHIFT_225, SW74 RSHIFT_175, SW75 FN_100, SW8 7, SW9 8, U1 STM32F072-LQFP48, U2 USBLC6-2SC6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

Commit message: PCB1
Parts:
- removed SW61: LCTRL_125, acheron_MX_SolderMask:MX125, symbol acheronSymbols:MXSwitch
- added D64, D66, D67, D68: 1N4148, acheron_Components:D_SOD-123, symbol doddle60-rescue:D-Device
- added SW66: SPACE_275, acheron_MX_SolderMask:MX275R, symbol acheronSymbols:MXSwitch
- added SW76: 150U_BKSLH, acheron_MX_SolderMask:MX150, symbol acheronSymbols:MXSwitch
- added SW77: ANSI_Enter, acheron_MX_SolderMask:MX225, symbol acheronSymbols:MXSwitch
- added SW78: BKSLSH_1U, acheron_MX_SolderMask:MX100, symbol acheronSymbols:MXSwitch
- added SW79: RSHIFT_1.75, acheron_MX_SolderMask:MX175, symbol acheronSymbols:MXSwitch
- added SW80, SW89: HENKAN_125, acheron_MX_SolderMask:MX125, symbol acheronSymbols:MXSwitch
- added SW81: MUHENKAN_125, acheron_MX_SolderMask:MX125, symbol acheronSymbols:MXSwitch
- added SW82, SW83: RALT_125, acheron_MX_SolderMask:MX125, symbol acheronSymbols:MXSwitch
- added SW84: RGUI_100, acheron_MX_SolderMask:MX100, symbol acheronSymbols:MXSwitch
- added SW85: RCTRL_125, acheron_MX_SolderMask:MX125, symbol acheronSymbols:MXSwitch
- added SW86: KANA_100, acheron_MX_SolderMask:MX100, symbol acheronSymbols:MXSwitch
- CB1, CB10, CB2, CB3, CB4, CB5, CB6, CB7, CB8, CB9, CRST1, CRST2, CSH1, CSH2, CSI1, CSO1, CUSB1: symbol Device:C_Small -> doddle60-rescue:C_Small-Device
- D1, D10, D11, D12, D13, D14, D15, D16, D17, D18, D19, D2, D20, D21, D22, D23, D24, D25, D26, D27, D28, D29, D3, D30, D31, D32, D33, D34, D35, D36, D37, D38, D39, D4, D40, D41, D42, D43, D44, D45, D46, D47, D48, D49, D5, D50, D51, D52, D53, D54, D55, D56, D57, D58, D59, D6, D60, D61, D62, D63, D65, D7, D8, D9: symbol Device:D -> doddle60-rescue:D-Device
- DF1: symbol Device:D_TVS -> doddle60-rescue:D_TVS-Device
- DL1: symbol Device:LED_Small -> doddle60-rescue:LED_Small-Device
- DRST1, DS1, DSH1: symbol Device:D_Schottky -> doddle60-rescue:D_Schottky-Device
- F1: symbol Device:Polyfuse_Small -> doddle60-rescue:Polyfuse_Small-Device
- G1, G2, G3, G4, G5, H1, H10, H2, H3, H4, H5, H6, H7, H9: symbol Mechanical:MountingHole -> doddle60-rescue:MountingHole-Mechanical
- H8: symbol Mechanical:MountingHole_Pad -> doddle60-rescue:MountingHole_Pad-Mechanical
- J2: symbol Connector_Generic:Conn_01x14 -> doddle60-rescue:Conn_01x14-Connector_Generic
- J3: symbol Connector:Conn_ARM_JTAG_SWD_10 -> doddle60-rescue:Conn_ARM_JTAG_SWD_10-Connector
- L2, L3: symbol Device:L_Core_Ferrite -> doddle60-rescue:L_Core_Ferrite-Device
- QRST1: symbol Transistor_BJT:DTC123J -> doddle60-rescue:DTC123J-Transistor_BJT
- RCC1, RCC2, RL1, RPU1, RRST1, RSH1, RSH2, RSI1, RSO1, RVDD1: symbol Device:R_Small -> doddle60-rescue:R_Small-Device
- SW54: value LCTRL_150 -> LCTRL_125; footprint acheron_MX_SolderMask:MX150 -> acheron_MX_SolderMask:MX125
- SW55: value LGUI_100 -> LGUI_125; footprint acheron_MX_SolderMask:MX100 -> acheron_MX_SolderMask:MX125
- SW56: value LALT_150 -> LALT_125; footprint acheron_MX_SolderMask:MX150 -> acheron_MX_SolderMask:MX125
- SW57: value SPACE_700 -> SPACE_275; footprint acheron_MX_SolderMask:MX700R -> acheron_MX_SolderMask:MX275R
- SW58: value RALT_150 -> RALT_125; footprint acheron_MX_SolderMask:MX150 -> acheron_MX_SolderMask:MX125
- SW59: value RGUI_100 -> RGUI_125; footprint acheron_MX_SolderMask:MX100 -> acheron_MX_SolderMask:MX125
- SW60: value RCTRL_150 -> RCTRL_125; footprint acheron_MX_SolderMask:MX150 -> acheron_MX_SolderMask:MX125
- SW61: renamed from SW62; value LGUI_125 -> LGUI_100; footprint acheron_MX_SolderMask:MX125 -> acheron_MX_SolderMask:MX100
- SW67: value SPACE_625 -> MUHENKAN_100; footprint acheron_MX_SolderMask:MX625R -> acheron_MX_SolderMask:MX100
- SW69: value RGUI_125 -> SPACE_125
- SW70: value FN_125 -> SPACE_450; footprint acheron_MX_SolderMask:MX125 -> acheron_MX_SolderMask:MX100
- SW71: value RCTRL_125 -> SPACE_225; footprint acheron_MX_SolderMask:MX125 -> acheron_MX_SolderMask:MX225R
- SW72: footprint acheron_MX_SolderMask:MX275 -> acheron_MX_SolderMask:MX275R
- SW73: footprint acheron_MX_SolderMask:MX225 -> acheron_MX_SolderMask:MX225R
- SWRST1: symbol Switch:SW_Push -> doddle60-rescue:SW_Push-Switch
- U2: symbol Power_Protection:USBLC6-2SC6 -> doddle60-rescue:USBLC6-2SC6-Power_Protection
- U3: symbol Regulator_Linear:MCP1700-3302E_SOT23 -> doddle60-rescue:MCP1700-3302E_SOT23-Regulator_Linear
- renumbered SW66 to SW62
Connections:
- net labels added: Col15
- wire segments 449 -> 498
Other:
- moved on the sheet: J1, L1, SW54, SW56, SW57, SW61, SW62, SW68, U1

Commit message: cache
Parts:
- removed SW66: SPACE_275, acheron_MX_SolderMask:MX275R, symbol acheronSymbols:MXSwitch
- removed SW69: SPACE_125, acheron_MX_SolderMask:MX125, symbol acheronSymbols:MXSwitch
- removed SW71: SPACE_225, acheron_MX_SolderMask:MX225R, symbol acheronSymbols:MXSwitch
- removed SW85: RCTRL_125, acheron_MX_SolderMask:MX125, symbol acheronSymbols:MXSwitch
Connections:
- net Col7: now also SW70.1 (Col)
- net Col8: now also SW86.1 (Col); no longer SW80.1 (Col)
- net Col9: now also SW80.1 (Col); no longer SW86.1 (Col)
- net at D66.2 (A), SW89.2 (Row): now also SW86.2 (Row); no longer SW80.2 (Row)
- net at D67.2 (A): now also SW80.2 (Row); no longer SW86.2 (Row)
Other:
- moved on the sheet: SW80, SW86
Changed lines of the file:
@@
 Connection ~ 6350 6250
-$Comp
-L acheronSymbols:MXSwitch SW66
-U 1 1 604F6338
-P 6350 8375
-F 0 "SW66" H 6350 8425 50  0000 C CNN
-F 1 "SPACE_275" H 6350 8300 40  0000 C CNN
-F 2 "acheron_MX_SolderMask:MX275R" H 6350 8375 50  0001 C CNN
-F 3 "" H 6350 8375 50  0001 C CNN
-	1    6350 8375
-	1    0    0    -1
-$EndComp
 $Comp
 L doddle60-rescue:D-Device D66
@@
 $EndComp
 Wire Wire Line
-	9750 8100 9750 8975
-Wire Wire Line
 	9350 8975 9350 9075
 Wire Wire Line
@@
 $EndComp
 Wire Wire Line
-	9350 8100 9750 8100
-$Comp
-L acheronSymbols:MXSwitch SW69
-U 1 1 6018A222
-P 9350 8450
-F 0 "SW69" H 9350 8500 50  0000 C CNN
-F 1 "SPACE_125" H 9350 8375 40  0000 C CNN
-F 2 "acheron_MX_SolderMask:MX125" H 9350 8450 50  0001 C CNN
-F 3 "" H 9350 8450 50  0001 C CNN
-	1    9350 8450
-	1    0    0    -1
-$EndComp
-Wire Wire Line
 	8850 5625 8850 6600
 Connection ~ 9350 6250
@@
 L acheronSymbols:MXSwitch SW86
 U 1 1 60A7E6F2
-P 11350 6600
-F 0 "SW86" H 11350 6650 50  0000 C CNN
-F 1 "KANA_100" H 11350 6525 40  0000 C CNN
-F 2 "acheron_MX_SolderMask:MX100" H 11350 6600 50  0001 C CNN
-F 3 "" H 11350 6600 50  0001 C CNN
-	1    11350 6600
+P 10350 9425
+F 0 "SW86" H 10350 9475 50  0000 C CNN
+F 1 "KANA_100" H 10350 9350 40  0000 C CNN
+F 2 "acheron_MX_SolderMask:MX100" H 10350 9425 50  0001 C CNN
+F 3 "" H 10350 9425 50  0001 C CNN
+	1    10350 9425
 	1    0    0    -1
 $EndComp
@@
 Wire Wire Line
 	6750 7200 6750 6250
-$Comp
-L acheronSymbols:MXSwitch SW71
-U 1 1 60A7E6E7
-P 10350 8450
-F 0 "SW71" H 10350 8500 50  0000 C CNN
-F 1 "SPACE_225" H 10350 8375 40  0000 C CNN
-F 2 "acheron_MX_SolderMask:MX225R" H 10350 8450 50  0001 C CNN
-F 3 "" H 10350 8450 50  0001 C CNN
-	1    10350 8450
-	1    0    0    -1
-$EndComp
 Wire Wire Line
 	10750 6250 10350 6250
@@
 L acheronSymbols:MXSwitch SW80
 U 1 1 60A7E6C5
-P 10350 9425
-F 0 "SW80" H 10350 9475 50  0000 C CNN
-F 1 "HENKAN_125" H 10350 9350 40  0000 C CNN
-F 2 "acheron_MX_SolderMask:MX125" H 10350 9425 50  0001 C CNN
-F 3 "" H 10350 9425 50  0001 C CNN
-	1    10350 9425
+P 11350 6600
+F 0 "SW80" H 11350 6650 50  0000 C CNN
+F 1 "HENKAN_125" H 11350 6525 40  0000 C CNN
+F 2 "acheron_MX_SolderMask:MX125" H 11350 6600 50  0001 C CNN
+F 3 "" H 11350 6600 50  0001 C CNN
+	1    11350 6600
 	1    0    0    -1
 $EndComp
@@
 	1    0    0    -1
 $EndComp
-Wire Wire Line
-	16000 9325 15850 9325
-$Comp
-L acheronSymbols:MXSwitch SW85
-U 1 1 61D8D563
-P 16350 9325
-F 0 "SW85" H 16350 9375 50  0000 C CNN
-F 1 "RCTRL_125" H 16350 9250 40  0000 C CNN
-F 2 "acheron_MX_SolderMask:MX125" H 16350 9325 50  0001 C CNN
-F 3 "" H 16350 9325 50  0001 C CNN
-	1    16350 9325
-	1    0    0    -1
-$EndComp
 $Comp
 L acheronSymbols:MXSwitch SW83
@@
 Wire Wire Line
 	6700 8025 6350 8025
-Connection ~ 6350 8025
 Wire Wire Line
 	3850 6600 3850 9425
@@
 	5850 6600 6000 6600
 Connection ~ 5850 5625
-Wire Wire Line
-	5850 6600 5850 8375
-Wire Wire Line
-	5850 8375 6000 8375
 Connection ~ 5850 6600
 Wire Wire Line
-	5850 8375 5850 9425
-Wire Wire Line
 	5850 9425 6000 9425
-Connection ~ 5850 8375
-Wire Wire Line
-	8850 8450 9000 8450
-Wire Wire Line
-	8850 8450 8850 9425
 Wire Wire Line
 	8850 9425 9000 9425
@@
 	9850 6600 10000 6600
 Connection ~ 9850 5625
-Wire Wire Line
-	9850 8450 10000 8450
-Wire Wire Line
-	9850 8450 9850 9425
 Wire Wire Line
 	9850 9425 10000 9425
@@
 $EndComp
 Wire Wire Line
-	16350 8975 16350 8500
-Wire Wire Line
-	16350 8500 16700 8500
-Wire Wire Line
 	6350 5950 9350 5950
-Connection ~ 9750 8100
-Wire Wire Line
-	9750 6250 9750 8100
 Wire Wire Line
 	10350 8100 10350 7750
@@
 Wire Wire Line
 	10750 6250 10750 7750
-Connection ~ 10350 8100
 Wire Wire Line
 	11350 5950 13350 5950
-Wire Wire Line
-	9850 6600 9850 8450
 Connection ~ 9850 6600
-Connection ~ 9850 8450
 Wire Wire Line
 	12850 6600 12850 9325
@@
 Connection ~ 14850 6600
 Wire Wire Line
-	15850 6600 15850 9325
-Connection ~ 15850 6600
-Wire Wire Line
 	13350 6250 13750 6250
 Wire Wire Line
@@
 	15750 6250 15750 8500
 Wire Wire Line
-	16700 6250 16700 8500
-Wire Wire Line
 	4300 8750 4300 9075
+Connection ~ 8850 6600
+Wire Wire Line
+	9750 6250 9750 8975
+Wire Wire Line
+	9850 6600 9850 9425
+Wire Wire Line
+	8850 6600 8850 9425
+Wire Wire Line
+	5850 6600 5850 9425
 $EndSCHEMATC
